File: Full_PCB.sch (KiCad schematic (older format))
At the start: 7 parts

Commit message: Small modifications to SCH
Connections:
- wire segments 49 -> 50
Changed lines of the file:
@@
 Text GLabel 4250 3700 0    60   Input ~ 0
-B-
-Text GLabel 5375 2300 2    60   Input ~ 0
 B-
 Text GLabel 5375 1925 2    60   Input ~ 0
@@
 	5375 1525 5950 1525
 Wire Wire Line
-	5950 1525 5950 2875
+	5950 1425 5950 2875
 Wire Wire Line
 	5950 2875 6150 2875
@@
 Text GLabel 4050 2600 2    60   Input ~ 0
 I_3_Boost
+Wire Wire Line
+	5950 1425 7250 1425
+Connection ~ 5950 1525
 $EndSCHEMATC
