File: PCB_Design/Bottom_side/5VBuck.sch (KiCad schematic (older format))
At the start: 11 parts, among them U5 TPS54302

Commit message: PCB bottom layer populated
PCB bottom layer populated, and waiting for top layer to be merged.
Changed lines of the file:
@@
 LIBS:contrib
 LIBS:valves
-LIBS:Custom_Library
 LIBS:Bottom_side-cache
 EELAYER 25 0
@@
 $Descr A4 11693 8268
 encoding utf-8
-Sheet 19 25
+Sheet 18 26
 Title ""
 Date ""
@@
 AR Path="/5A57B54F/5A5E496B/5A5E4AD0" Ref="U5"  Part="1"
 AR Path="/5A57B54F/5A5E5DCC/5A5E4AD0" Ref="U6"  Part="1"
-F 0 "U5" H 4900 3400 60  0000 C CNN
+F 0 "U6" H 4900 3400 60  0000 C CNN
 F 1 "TPS54302" H 4900 3300 60  0000 C CNN
 F 2 "TO_SOT_Packages_SMD:SOT-23-6_Handsoldering" H 4900 3400 60  0001 C CNN
@@
 AR Path="/5A57B54F/5A5E496B/5A5E4AD1" Ref="CVCCbuck1"  Part="1"
 AR Path="/5A57B54F/5A5E5DCC/5A5E4AD1" Ref="CVCCbuck2"  Part="1"
-F 0 "CVCCbuck1" H 4025 3500 50  0000 L CNN
+F 0 "CVCCbuck2" H 4025 3500 50  0000 L CNN
 F 1 "10u" H 4025 3300 50  0000 L CNN
 F 2 "Capacitors_SMD:C_0603" H 4038 3250 50  0001 C CNN
@@
 AR Path="/5A57B54F/5A5E496B/5A5E4AD2" Ref="Cboot1"  Part="1"
 AR Path="/5A57B54F/5A5E5DCC/5A5E4AD2" Ref="Cboot2"  Part="1"
-F 0 "Cboot1" H 5625 3500 50  0000 L CNN
+F 0 "Cboot2" H 5625 3500 50  0000 L CNN
 F 1 ".1uF" H 5625 3300 50  0000 L CNN
 F 2 "Capacitors_SMD:C_0805" H 5638 3250 50  0001 C CNN
@@
 AR Path="/5A57B54F/5A5E496B/5A5E4AD3" Ref="5V_ind1"  Part="1"
 AR Path="/5A57B54F/5A5E5DCC/5A5E4AD3" Ref="5V_ind2"  Part="1"
-F 0 "5V_ind1" V 5950 3550 50  0000 C CNN
+F 0 "5V_ind2" V 5950 3550 50  0000 C CNN
 F 1 "10u" V 6075 3550 50  0000 C CNN
 F 2 "Inductors_SMD:L_10.4x10.4_H4.8" H 6000 3550 50  0001 C CNN
@@
 AR Path="/5A57B54F/5A5E496B/5A5E4AD4" Ref="R_fb_hi1"  Part="1"
 AR Path="/5A57B54F/5A5E5DCC/5A5E4AD4" Ref="R_fb_hi2"  Part="1"
-F 0 "R_fb_hi1" V 6380 3700 50  0000 C CNN
+F 0 "R_fb_hi2" V 6380 3700 50  0000 C CNN
 F 1 "R" V 6300 3700 50  0000 C CNN
 F 2 "Resistors_SMD:R_0603" V 6230 3700 50  0001 C CNN
@@
 AR Path="/5A57B54F/5A5E496B/5A5E4AD5" Ref="R_fb_lo1"  Part="1"
 AR Path="/5A57B54F/5A5E5DCC/5A5E4AD5" Ref="R_fb_lo2"  Part="1"
-F 0 "R_fb_lo1" V 6380 4100 50  0000 C CNN
+F 0 "R_fb_lo2" V 6380 4100 50  0000 C CNN
 F 1 "R" V 6300 4100 50  0000 C CNN
 F 2 "Resistors_SMD:R_0603" V 6230 4100 50  0001 C CNN
@@
 AR Path="/5A57B54F/5A5E496B/5A5E4AD6" Ref="CBulk1"  Part="1"
 AR Path="/5A57B54F/5A5E5DCC/5A5E4AD6" Ref="CBulk3"  Part="1"
-F 0 "CBulk1" H 6450 3900 50  0000 L CNN
+F 0 "CBulk3" H 6450 3900 50  0000 L CNN
 F 1 "C" H 6625 3600 50  0000 L CNN
 F 2 "Capacitors_Tantalum_SMD:CP_Tantalum_Case-C_EIA-6032-28_Hand" H 6638 3550 50  0001 C CNN
@@
 AR Path="/5A57B54F/5A5E496B/5A5E4AD7" Ref="CBulk2"  Part="1"
 AR Path="/5A57B54F/5A5E5DCC/5A5E4AD7" Ref="CBulk4"  Part="1"
-F 0 "CBulk2" H 6750 3900 50  0000 L CNN
+F 0 "CBulk4" H 6750 3900 50  0000 L CNN
 F 1 "C" H 6825 3600 50  0000 L CNN
 F 2 "Capacitors_Tantalum_SMD:CP_Tantalum_Case-C_EIA-6032-28_Hand" H 6838 3550 50  0001 C CNN
@@
 $EndComp
 $Comp
-L GND #PWR055
+L GND #PWR061
 U 1 1 5A5E4AD8
 P 6600 4350
-AR Path="/5A57B54F/5A5E496B/5A5E4AD8" Ref="#PWR055"  Part="1"
-AR Path="/5A57B54F/5A5E5DCC/5A5E4AD8" Ref="#PWR060"  Part="1"
-F 0 "#PWR060" H 6600 4100 50  0001 C CNN
+AR Path="/5A57B54F/5A5E496B/5A5E4AD8" Ref="#PWR061"  Part="1"
+AR Path="/5A57B54F/5A5E5DCC/5A5E4AD8" Ref="#PWR066"  Part="1"
+F 0 "#PWR066" H 6600 4100 50  0001 C CNN
 F 1 "GND" H 6600 4200 50  0000 C CNN
 F 2 "" H 6600 4350 50  0001 C CNN
@@
 $EndComp
 $Comp
-L GND #PWR056
+L GND #PWR062
 U 1 1 5A5E4AD9
 P 6300 4350
-AR Path="/5A57B54F/5A5E496B/5A5E4AD9" Ref="#PWR056"  Part="1"
-AR Path="/5A57B54F/5A5E5DCC/5A5E4AD9" Ref="#PWR061"  Part="1"
-F 0 "#PWR061" H 6300 4100 50  0001 C CNN
+AR Path="/5A57B54F/5A5E496B/5A5E4AD9" Ref="#PWR062"  Part="1"
+AR Path="/5A57B54F/5A5E5DCC/5A5E4AD9" Ref="#PWR067"  Part="1"
+F 0 "#PWR067" H 6300 4100 50  0001 C CNN
 F 1 "GND" H 6300 4200 50  0000 C CNN
 F 2 "" H 6300 4350 50  0001 C CNN
@@
 $EndComp
 $Comp
-L GND #PWR057
+L GND #PWR063
 U 1 1 5A5E4ADA
 P 6800 4350
-AR Path="/5A57B54F/5A5E496B/5A5E4ADA" Ref="#PWR057"  Part="1"
-AR Path="/5A57B54F/5A5E5DCC/5A5E4ADA" Ref="#PWR062"  Part="1"
-F 0 "#PWR062" H 6800 4100 50  0001 C CNN
+AR Path="/5A57B54F/5A5E496B/5A5E4ADA" Ref="#PWR063"  Part="1"
+AR Path="/5A57B54F/5A5E5DCC/5A5E4ADA" Ref="#PWR068"  Part="1"
+F 0 "#PWR068" H 6800 4100 50  0001 C CNN
 F 1 "GND" H 6800 4200 50  0000 C CNN
 F 2 "" H 6800 4350 50  0001 C CNN
@@
 Connection ~ 6800 3550
 $Comp
-L GND #PWR058
+L GND #PWR064
 U 1 1 5A5E4ADE
 P 4200 3550
-AR Path="/5A57B54F/5A5E496B/5A5E4ADE" Ref="#PWR058"  Part="1"
-AR Path="/5A57B54F/5A5E5DCC/5A5E4ADE" Ref="#PWR063"  Part="1"
-F 0 "#PWR063" H 4200 3300 50  0001 C CNN
+AR Path="/5A57B54F/5A5E496B/5A5E4ADE" Ref="#PWR064"  Part="1"
+AR Path="/5A57B54F/5A5E5DCC/5A5E4ADE" Ref="#PWR069"  Part="1"
+F 0 "#PWR069" H 4200 3300 50  0001 C CNN
 F 1 "GND" H 4200 3400 50  0000 C CNN
 F 2 "" H 4200 3550 50  0001 C CNN
@@
 AR Path="/5A57B54F/5A5E496B/5A5E4EB0" Ref="R_en_div_high1"  Part="1"
 AR Path="/5A57B54F/5A5E5DCC/5A5E4EB0" Ref="R_en_div_high2"  Part="1"
-F 0 "R_en_div_high1" V 3750 4000 50  0000 C CNN
+F 0 "R_en_div_high2" V 3750 4000 50  0000 C CNN
 F 1 "R" V 3850 3900 50  0000 C CNN
 F 2 "Resistors_SMD:R_0603" V 3780 3900 50  0001 C CNN
@@
 AR Path="/5A57B54F/5A5E496B/5A5E50C3" Ref="R_en_div_low1"  Part="1"
 AR Path="/5A57B54F/5A5E5DCC/5A5E50C3" Ref="R_en_div_low2"  Part="1"
-F 0 "R_en_div_low1" V 4050 4200 50  0000 C CNN
+F 0 "R_en_div_low2" V 4050 4200 50  0000 C CNN
 F 1 "R" V 3850 4300 50  0000 C CNN
 F 2 "Resistors_SMD:R_0603" V 3780 4300 50  0001 C CNN
@@
 	3850 4450 3850 4550
 $Comp
-L GND #PWR059
+L GND #PWR065
 U 1 1 5A5E5227
 P 3850 4550
-AR Path="/5A57B54F/5A5E496B/5A5E5227" Ref="#PWR059"  Part="1"
-AR Path="/5A57B54F/5A5E5DCC/5A5E5227" Ref="#PWR064"  Part="1"
-F 0 "#PWR064" H 3850 4300 50  0001 C CNN
+AR Path="/5A57B54F/5A5E496B/5A5E5227" Ref="#PWR065"  Part="1"
+AR Path="/5A57B54F/5A5E5DCC/5A5E5227" Ref="#PWR070"  Part="1"
+F 0 "#PWR070" H 3850 4300 50  0001 C CNN
 F 1 "GND" H 3850 4400 50  0000 C CNN
 F 2 "" H 3850 4550 50  0001 C CNN
@@
 AR Path="/5A57B54F/5A5E496B/5A5E5285" Ref="R_enable1"  Part="1"
 AR Path="/5A57B54F/5A5E5DCC/5A5E5285" Ref="R_enable2"  Part="1"
-F 0 "R_enable1" V 3580 4250 50  0000 C CNN
+F 0 "R_enable2" V 3580 4250 50  0000 C CNN
 F 1 "R" V 3500 4250 50  0000 C CNN
 F 2 "Resistors_SMD:R_0603" V 3430 4250 50  0001 C CNN
