File: PCB_Design/Bottom_side/INA_5V_OUT.sch (KiCad schematic (older format))
At the start: 4 parts

Commit message: Updated PCB structure tree
Full_PCB now includes bottom and top layer hierarchical sheets
Changed lines of the file:
@@
 LIBS:power
 LIBS:device
-LIBS:switches
-LIBS:relays
-LIBS:motors
 LIBS:transistors
 LIBS:conn
@@
 LIBS:contrib
 LIBS:valves
-LIBS:Bottom_side-cache
+LIBS:Full_PCB-cache
 EELAYER 25 0
 EELAYER END
 $Descr A4 11693 8268
 encoding utf-8
-Sheet 21 26
+Sheet 20 26
 Title "INA139 & Voltage Divider for Voltage Measurement"
 Date "2017-06-14"
@@
 AR Path="/5A57B54F/5A5E7CAE/5A5E5F13" Ref="R11"  Part="1"
 AR Path="/5A57B54F/5A5E7CB4/5A5E5F13" Ref="R12"  Part="1"
-F 0 "R12" V 2580 1750 50  0000 C CNN
+F 0 "R11" V 2580 1750 50  0000 C CNN
 F 1 "100k" V 2500 1750 50  0000 C CNN
 F 2 "Resistors_SMD:R_0603" V 2430 1750 50  0001 C CNN
@@
 AR Path="/5A57B54F/5A5E7CAE/5A5E5F14" Ref="20m9"  Part="1"
 AR Path="/5A57B54F/5A5E7CB4/5A5E5F14" Ref="20m10"  Part="1"
-F 0 "20m10" V 3430 2250 50  0000 C CNN
+F 0 "20m9" V 3430 2250 50  0000 C CNN
 F 1 "R_Shunt" V 3350 2250 50  0000 C CNN
 F 2 "Resistors_SMD:R_0805" V 3280 2250 50  0001 C CNN
@@
 AR Path="/5A57B54F/5A5E7CAE/5A5E5F15" Ref="C_Bypass9"  Part="1"
 AR Path="/5A57B54F/5A5E7CB4/5A5E5F15" Ref="C_Bypass10"  Part="1"
-F 0 "C_Bypass10" H 4025 1850 50  0000 L CNN
+F 0 "C_Bypass9" H 4025 1850 50  0000 L CNN
 F 1 ".1u" H 4025 1650 50  0000 L CNN
 F 2 "Capacitors_SMD:C_0603" H 4038 1600 50  0001 C CNN
@@
 Connection ~ 4000 1550
 $Comp
-L GND #PWR074
+L GND #PWR067
 U 1 1 5A5E5F16
 P 4000 1900
-AR Path="/5A57B54F/5A5E7852/5A5E5F16" Ref="#PWR074"  Part="1"
-AR Path="/5A57B54F/5A5E5DCE/5A5E5F16" Ref="#PWR071"  Part="1"
-AR Path="/5A57B54F/5A5E7CAE/5A5E5F16" Ref="#PWR077"  Part="1"
-AR Path="/5A57B54F/5A5E7CB4/5A5E5F16" Ref="#PWR080"  Part="1"
-F 0 "#PWR080" H 4000 1650 50  0001 C CNN
+AR Path="/5A57B54F/5A5E7852/5A5E5F16" Ref="#PWR067"  Part="1"
+AR Path="/5A57B54F/5A5E5DCE/5A5E5F16" Ref="#PWR064"  Part="1"
+AR Path="/5A57B54F/5A5E7CAE/5A5E5F16" Ref="#PWR070"  Part="1"
+AR Path="/5A57B54F/5A5E7CB4/5A5E5F16" Ref="#PWR073"  Part="1"
+F 0 "#PWR070" H 4000 1650 50  0001 C CNN
 F 1 "GND" H 4000 1750 50  0000 C CNN
 F 2 "" H 4000 1900 50  0001 C CNN
@@
 $EndComp
 $Comp
-L GND #PWR075
+L GND #PWR068
 U 1 1 5A5E5F17
 P 2900 1750
-AR Path="/5A57B54F/5A5E7852/5A5E5F17" Ref="#PWR075"  Part="1"
-AR Path="/5A57B54F/5A5E5DCE/5A5E5F17" Ref="#PWR072"  Part="1"
-AR Path="/5A57B54F/5A5E7CAE/5A5E5F17" Ref="#PWR078"  Part="1"
-AR Path="/5A57B54F/5A5E7CB4/5A5E5F17" Ref="#PWR081"  Part="1"
-F 0 "#PWR081" H 2900 1500 50  0001 C CNN
+AR Path="/5A57B54F/5A5E7852/5A5E5F17" Ref="#PWR068"  Part="1"
+AR Path="/5A57B54F/5A5E5DCE/5A5E5F17" Ref="#PWR065"  Part="1"
+AR Path="/5A57B54F/5A5E7CAE/5A5E5F17" Ref="#PWR071"  Part="1"
+AR Path="/5A57B54F/5A5E7CB4/5A5E5F17" Ref="#PWR074"  Part="1"
+F 0 "#PWR071" H 2900 1500 50  0001 C CNN
 F 1 "GND" H 2900 1600 50  0000 C CNN
 F 2 "" H 2900 1750 50  0001 C CNN
@@
 AR Path="/5A57B54F/5A5E7CAE/5A5E5F18" Ref="INA9"  Part="1"
 AR Path="/5A57B54F/5A5E7CB4/5A5E5F18" Ref="INA10"  Part="1"
-F 0 "INA10" H 3350 1475 60  0000 C CNN
+F 0 "INA9" H 3350 1475 60  0000 C CNN
 F 1 "INA139" H 3350 2025 60  0000 C CNN
 F 2 "TO_SOT_Packages_SMD:SOT-23-5" H 3225 1800 60  0001 C CNN
@@
 I_out
 $Comp
-L GND #PWR076
+L GND #PWR069
 U 1 1 5A5E5F19
 P 2500 1900
-AR Path="/5A57B54F/5A5E7852/5A5E5F19" Ref="#PWR076"  Part="1"
-AR Path="/5A57B54F/5A5E5DCE/5A5E5F19" Ref="#PWR073"  Part="1"
-AR Path="/5A57B54F/5A5E7CAE/5A5E5F19" Ref="#PWR079"  Part="1"
-AR Path="/5A57B54F/5A5E7CB4/5A5E5F19" Ref="#PWR082"  Part="1"
-F 0 "#PWR082" H 2500 1650 50  0001 C CNN
+AR Path="/5A57B54F/5A5E7852/5A5E5F19" Ref="#PWR069"  Part="1"
+AR Path="/5A57B54F/5A5E5DCE/5A5E5F19" Ref="#PWR066"  Part="1"
+AR Path="/5A57B54F/5A5E7CAE/5A5E5F19" Ref="#PWR072"  Part="1"
+AR Path="/5A57B54F/5A5E7CB4/5A5E5F19" Ref="#PWR075"  Part="1"
+F 0 "#PWR072" H 2500 1650 50  0001 C CNN
 F 1 "GND" H 2500 1750 50  0000 C CNN
 F 2 "" H 2500 1900 50  0001 C CNN
