File: PCB_Design/Bottom_side/SWITCH.sch (KiCad schematic (older format))
At the start: 13 parts, among them Q5 Q_PMOS_GSD, Q6 Q_PMOS_GSD, Q7 Q_PMOS_GSD, Q8 Q_NMOS_GSD, Q9 Q_NMOS_GSD

Commit message: PCB bottom layer populated
PCB bottom layer populated, and waiting for top layer to be merged.
Other:
- note added: "Dual switch for redundancy"
- note added: "First RBF switch cuts all power"
- note added: "MCU high impedance / high => ON\nMCU pull to ground => OFF"
- note added: "Second RBF switch cuts battery output"
- note added: "Two switches required by CubeSat standard safety requirements"
- note added: "Voltage divider\n3.6V max\nFor MCU safety"
- note removed: "MCU high impedance => ON\nMCU pull to ground => OFF"
- note removed: "No MCU control\nOnly RBF"
- note removed: "Optional diode\n"
- note removed: "Voltage divider\n3.6V max"
Changed lines of the file:
@@
 LIBS:contrib
 LIBS:valves
-LIBS:Custom_Library
 LIBS:Bottom_side-cache
 EELAYER 25 0
@@
 $Descr A4 11693 8268
 encoding utf-8
-Sheet 16 25
+Sheet 16 26
 Title ""
 Date ""
@@
 	0    1    1    0
 $EndComp
-Text Notes 2900 2350 0    60   ~ 0
-Optional diode\n
 Text Notes 3850 3300 0    60   ~ 0
 THESE TWO SWITCHES \nCAN BE CONTROLLED BY MCU
@@
 	0    1    1    0
 $EndComp
-Text Notes 2750 2900 0    60   ~ 0
-No MCU control\nOnly RBF
+Text Notes 1900 1500 0    60   ~ 0
+First RBF switch cuts all power
 Wire Wire Line
 	4300 2500 4100 2500
@@
 	4500 950  4500 800
 Text Notes 4950 1900 0    60   ~ 0
-MCU high impedance => ON\nMCU pull to ground => OFF
+MCU high impedance / high => ON\nMCU pull to ground => OFF
 $Comp
 L R RDivLo1
@@
 Connection ~ 3500 1800
 $Comp
-L GND #PWR053
+L GND #PWR059
 U 1 1 5A584A02
 P 4250 1800
-F 0 "#PWR053" H 4250 1550 50  0001 C CNN
+F 0 "#PWR059" H 4250 1550 50  0001 C CNN
 F 1 "GND" H 4250 1650 50  0000 C CNN
 F 2 "" H 4250 1800 50  0001 C CNN
@@
 	4800 1700 4800 1550
 Connection ~ 3900 1800
-Text Notes 3650 1650 0    60   ~ 0
-Voltage divider\n3.6V max
+Text Notes 3650 1550 0    60   ~ 0
+Voltage divider\n3.6V max\nFor MCU safety
 Text HLabel 2200 2500 0    60   Input ~ 0
 Vin
@@
 $EndComp
 $Comp
-L GND #PWR054
+L GND #PWR060
 U 1 1 5A70AB37
 P 3750 4150
-F 0 "#PWR054" H 3750 3900 50  0001 C CNN
+F 0 "#PWR060" H 3750 3900 50  0001 C CNN
 F 1 "GND" H 3750 4000 50  0000 C CNN
 F 2 "" H 3750 4150 50  0001 C CNN
@@
 	3150 3650 3150 3800
 Connection ~ 3150 3800
+Text Notes 4150 3950 0    60   ~ 0
+Dual switch for redundancy
+Text Notes 3950 2300 0    60   ~ 0
+Two switches required by CubeSat standard safety requirements
+Text Notes 4650 950  0    60   ~ 0
+Second RBF switch cuts battery output
 $EndSCHEMATC

Commit message: Updated PCB structure tree
Full_PCB now includes bottom and top layer hierarchical sheets
Parts:
- removed 100k1, 1k1: R, Resistors_SMD:R_0603, symbol R
- removed Q5, Q6, Q7: Q_PMOS_GSD, TO_SOT_Packages_SMD:SOT-23, symbol Q_PMOS_GSD
- removed Q8, Q9: Q_NMOS_GSD, TO_SOT_Packages_SMD:SOT-23, symbol Q_NMOS_GSD
- added D4: D, Diodes_SMD:D_SMA, symbol D
- added PMOS1: PCH GDS, TO_SOT_Packages_SMD:TDSON-8-1, symbol Q_PMOS_GSD
- added PMOS2, PMOS3: Pch GDS, TO_SOT_Packages_SMD:TDSON-8-1, symbol Q_PMOS_GSD
- Nmos_sw1: footprint TO_SOT_Packages_SMD:SOT-23 -> TO_SOT_Packages_SMD:TDSON-8-1
Connections:
- net BATT+: now also D4.1 (K), PMOS2.2 (S)
- net RBF1: now also PMOS1.1 (G)
- net Vin: now also PMOS1.2 (S)
- net Vout: now also PMOS3.3 (D)
- net at Nmos_sw1.3 (D), R_pull1.1: now also PMOS2.1 (G), PMOS3.1 (G)
- new net: D4.2 (A), PMOS1.3 (D)
- new net: PMOS2.3 (D), PMOS3.2 (S)
Other:
- note added: "MCU POWER MUST NOT BE CONNECTED HERE"
- note added: "MCU high impedance => ON\nMCU pull to ground => OFF"
- note added: "No MCU control\nOnly RBF"
- note added: "Optional diode\n"
- note added: "PHYSICAL SWITCH TO GND"
- note added: "Power MCU from Batt+\n"
- note added: "Voltage divider\n3.6V max"
- note removed: "Dual switch for redundancy"
- note removed: "First RBF switch cuts all power"
- note removed: "GND before flight, FLOATING when activated"
- note removed: "MCU high impedance / high => ON\nMCU pull to ground => OFF"
- note removed: "Second RBF switch cuts battery output"
- note removed: "Two switches required by CubeSat standard safety requirements"
- note removed: "Voltage divider\n3.6V max\nFor MCU safety"
Changed lines of the file:
@@
 LIBS:power
 LIBS:device
-LIBS:switches
-LIBS:relays
-LIBS:motors
 LIBS:transistors
 LIBS:conn
@@
 LIBS:contrib
 LIBS:valves
-LIBS:Bottom_side-cache
+LIBS:Full_PCB-cache
 EELAYER 25 0
 EELAYER END
@@
 $EndDescr
 $Comp
+L D D4
+U 1 1 5A5849EF
+P 3300 2500
+F 0 "D4" H 3300 2600 50  0000 C CNN
+F 1 "D" H 3300 2400 50  0000 C CNN
+F 2 "Diodes_SMD:D_SMA" H 3300 2500 50  0001 C CNN
+F 3 "" H 3300 2500 50  0000 C CNN
+	1    3300 2500
+	-1   0    0    1
+$EndComp
+$Comp
+L Q_PMOS_GSD PMOS3
+U 1 1 5A5849F0
+P 4500 2400
+F 0 "PMOS3" V 4800 2400 50  0000 L CNN
+F 1 "Pch GDS" V 4700 2350 50  0000 L CNN
+F 2 "TO_SOT_Packages_SMD:TDSON-8-1" H 4700 2500 50  0001 C CNN
+F 3 "" H 4500 2400 50  0000 C CNN
+	1    4500 2400
+	0    1    1    0
+$EndComp
+$Comp
 L R R7
 U 1 1 5A5849F2
@@
 $EndComp
 $Comp
+L Q_PMOS_GSD PMOS1
+U 1 1 5A5849F3
+P 2750 2400
+F 0 "PMOS1" V 3050 2300 50  0000 L CNN
+F 1 "PCH GDS" V 2950 2200 50  0000 L CNN
+F 2 "TO_SOT_Packages_SMD:TDSON-8-1" H 2950 2500 50  0001 C CNN
+F 3 "" H 2750 2400 50  0000 C CNN
+	1    2750 2400
+	0    1    1    0
+$EndComp
+$Comp
 L Q_NMOS_GSD Nmos_sw1
 U 1 1 5A5849F4
@@
 F 0 "Nmos_sw1" H 4800 1600 50  0000 L CNN
 F 1 "Logic level Nch mosfet" H 3800 1350 50  0000 L CNN
-F 2 "TO_SOT_Packages_SMD:SOT-23" H 4800 1650 50  0001 C CNN
+F 2 "TO_SOT_Packages_SMD:TDSON-8-1" H 4800 1650 50  0001 C CNN
 F 3 "" H 4600 1550 50  0000 C CNN
 	1    4600 1550
@@
 	0    1    1    0
 $EndComp
-Text Notes 3850 3300 0    60   ~ 0
+Text Notes 2900 2350 0    60   ~ 0
+Optional diode\n
+Text Notes 3850 2950 0    60   ~ 0
 THESE TWO SWITCHES \nCAN BE CONTROLLED BY MCU
+Text Notes 3600 3800 0    60   ~ 0
+PHYSICAL SWITCH TO GND
+$Comp
+L Q_PMOS_GSD PMOS2
+U 1 1 5A5849FC
+P 3900 2400
+F 0 "PMOS2" V 4200 2350 50  0000 L CNN
+F 1 "Pch GDS" V 4100 2350 50  0000 L CNN
+F 2 "TO_SOT_Packages_SMD:TDSON-8-1" H 4100 2500 50  0001 C CNN
+F 3 "" H 3900 2400 50  0000 C CNN
+	1    3900 2400
+	0    1    1    0
+$EndComp
 $Comp
 L R R_pull1
@@
 	0    1    1    0
 $EndComp
-Text Notes 1900 1500 0    60   ~ 0
-First RBF switch cuts all power
+Text Notes 2750 2900 0    60   ~ 0
+No MCU control\nOnly RBF
 Wire Wire Line
 	4300 2500 4100 2500
 Wire Wire Line
-	2950 2500 3700 2500
+	3450 2500 3700 2500
+Wire Wire Line
+	3150 2500 2950 2500
 Wire Wire Line
 	2200 2500 2550 2500
@@
 	4500 950  4500 800
 Text Notes 4950 1900 0    60   ~ 0
-MCU high impedance / high => ON\nMCU pull to ground => OFF
+MCU high impedance => ON\nMCU pull to ground => OFF
 $Comp
 L R RDivLo1
@@
 Connection ~ 3500 1800
 $Comp
-L GND #PWR059
+L GND #PWR053
 U 1 1 5A584A02
 P 4250 1800
-F 0 "#PWR059" H 4250 1550 50  0001 C CNN
+F 0 "#PWR053" H 4250 1550 50  0001 C CNN
 F 1 "GND" H 4250 1650 50  0000 C CNN
 F 2 "" H 4250 1800 50  0001 C CNN
@@
 	4800 1700 4800 1550
 Connection ~ 3900 1800
-Text Notes 3650 1550 0    60   ~ 0
-Voltage divider\n3.6V max\nFor MCU safety
+Text Notes 3650 1650 0    60   ~ 0
+Voltage divider\n3.6V max
+Text Notes 5550 2650 0    60   ~ 0
+MCU POWER MUST NOT BE CONNECTED HERE
+Text Notes 3550 3150 0    60   ~ 0
+Power MCU from Batt+\n
 Text HLabel 2200 2500 0    60   Input ~ 0
 Vin
@@
 BATT-
 Wire Wire Line
-	3500 3300 3500 3600
-$Comp
-L Q_PMOS_GSD Q7
-U 1 1 5A6925D8
-P 4500 2400
-F 0 "Q7" H 4700 2450 50  0000 L CNN
-F 1 "Q_PMOS_GSD" H 4700 2350 50  0000 L CNN
-F 2 "TO_SOT_Packages_SMD:SOT-23" H 4700 2500 50  0001 C CNN
-F 3 "" H 4500 2400 50  0001 C CNN
-	1    4500 2400
-	0    1    1    0
-$EndComp
-$Comp
-L Q_PMOS_GSD Q6
-U 1 1 5A69265B
-P 3900 2400
-F 0 "Q6" H 4100 2450 50  0000 L CNN
-F 1 "Q_PMOS_GSD" H 4100 2350 50  0000 L CNN
-F 2 "TO_SOT_Packages_SMD:SOT-23" H 4100 2500 50  0001 C CNN
-F 3 "" H 3900 2400 50  0001 C CNN
-	1    3900 2400
-	0    1    1    0
-$EndComp
-$Comp
-L Q_PMOS_GSD Q5
-U 1 1 5A69268E
-P 2750 2400
-F 0 "Q5" H 2950 2450 50  0000 L CNN
-F 1 "Q_PMOS_GSD" H 2950 2350 50  0000 L CNN
-F 2 "TO_SOT_Packages_SMD:SOT-23" H 2950 2500 50  0001 C CNN
-F 3 "" H 2750 2400 50  0001 C CNN
-	1    2750 2400
-	0    1    1    0
-$EndComp
-$Comp
-L Q_NMOS_GSD Q8
-U 1 1 5A70AA86
-P 3400 3800
-F 0 "Q8" H 3600 3850 50  0000 L CNN
-F 1 "Q_NMOS_GSD" H 3600 3750 50  0000 L CNN
-F 2 "TO_SOT_Packages_SMD:SOT-23" H 3600 3900 50  0001 C CNN
-F 3 "" H 3400 3800 50  0001 C CNN
-	1    3400 3800
-	1    0    0    -1
-$EndComp
-$Comp
-L GND #PWR060
-U 1 1 5A70AB37
-P 3750 4150
-F 0 "#PWR060" H 3750 3900 50  0001 C CNN
-F 1 "GND" H 3750 4000 50  0000 C CNN
-F 2 "" H 3750 4150 50  0001 C CNN
-F 3 "" H 3750 4150 50  0001 C CNN
-	1    3750 4150
-	1    0    0    -1
-$EndComp
-Wire Wire Line
-	3500 4150 3500 4000
-Connection ~ 3200 2500
-$Comp
-L R 100k1
-U 1 1 5A70ABBE
-P 2900 3550
-F 0 "100k1" V 2980 3550 50  0000 C CNN
-F 1 "R" V 2900 3550 50  0000 C CNN
-F 2 "Resistors_SMD:R_0603" V 2830 3550 50  0001 C CNN
-F 3 "" H 2900 3550 50  0001 C CNN
-	1    2900 3550
-	1    0    0    -1
-$EndComp
-Wire Wire Line
-	3200 3800 2900 3800
-Wire Wire Line
-	2900 3700 2900 4050
-Wire Wire Line
-	2900 3400 2900 2950
-Wire Wire Line
-	2900 2950 3200 2950
-Wire Wire Line
-	3200 2950 3200 2500
-Connection ~ 2900 3800
-$Comp
-L R 1k1
-U 1 1 5A70AD73
-P 2900 4200
-F 0 "1k1" V 2980 4200 50  0000 C CNN
-F 1 "R" V 2900 4200 50  0000 C CNN
-F 2 "Resistors_SMD:R_0603" V 2830 4200 50  0001 C CNN
-F 3 "" H 2900 4200 50  0001 C CNN
-	1    2900 4200
-	1    0    0    -1
-$EndComp
-Text HLabel 2900 4500 2    60   Input ~ 0
+	3500 3300 3500 3550
+Text HLabel 3500 3550 2    60   Input ~ 0
 RBF_GND
-Wire Wire Line
-	2900 4500 2900 4350
-Text Notes 2350 4700 0    60   ~ 0
-GND before flight, FLOATING when activated
-Wire Wire Line
-	4100 4150 3500 4150
-Wire Wire Line
-	4100 3850 4100 4150
-Connection ~ 3750 4150
-$Comp
-L Q_NMOS_GSD Q9
-U 1 1 5A70C7AB
-P 4000 3650
-F 0 "Q9" H 4200 3700 50  0000 L CNN
-F 1 "Q_NMOS_GSD" H 4200 3600 50  0000 L CNN
-F 2 "TO_SOT_Packages_SMD:SOT-23" H 4200 3750 50  0001 C CNN
-F 3 "" H 4000 3650 50  0001 C CNN
-	1    4000 3650
-	1    0    0    -1
-$EndComp
-Wire Wire Line
-	4100 3450 4100 3400
-Wire Wire Line
-	4100 3400 3500 3400
-Connection ~ 3500 3400
-Wire Wire Line
-	3800 3650 3150 3650
-Wire Wire Line
-	3150 3650 3150 3800
-Connection ~ 3150 3800
-Text Notes 4150 3950 0    60   ~ 0
-Dual switch for redundancy
-Text Notes 3950 2300 0    60   ~ 0
-Two switches required by CubeSat standard safety requirements
-Text Notes 4650 950  0    60   ~ 0
-Second RBF switch cuts battery output
 $EndSCHEMATC
