File: EPS/Boost_converters.sch (KiCad schematic (older format))
At the start: 42 parts

Commit message: Updated schematics
Parts:
- removed R? (x3): R, symbol R
- added MAX5395? (x3): MAX5395, symbol MAX5395
- added R? (x3): R, symbol R
Connections:
- net FB1: now also MAX5395?.8 (H)
- net FB2: now also MAX5395?.8 (H)
- net FB3: now also MAX5395?.8 (H)
- net GND: now also MAX5395?.1 (L), MAX5395?.1 (L), MAX5395?.1 (L), MAX5395?.2 (gnd), MAX5395?.2 (gnd), MAX5395?.2 (gnd), MAX5395?.3 (ADDR0), R?.1, R?.1, R?.1
- new net: MAX5395?.7 (W), R?.2 (x3)
- new net 3V3: MAX5395?.3 (ADDR0), MAX5395?.6 (VDD), MAX5395?.6 (VDD), MAX5395?.6 (VDD)
- new net SCL: MAX5395?.5 (SCL), MAX5395?.5 (SCL), MAX5395?.5 (SCL)
- new net SDA: MAX5395?.4 (SDA), MAX5395?.4 (SDA), MAX5395?.4 (SDA)
- no-connect marks 0 -> 1
Other:
- note added: "Feedback resistors:\nHigh side 300k\nLow side 50k POT + 50k \nFull output voltage range 5V - 8.75V"
- note added: "MAX5395MATA+T is 50k version"
- note added: "Slave address 0101000"
- note added: "Slave address 0101001"
- note added: "Slave address 0101011"
- note removed: "Need values for capacitors,\nfeedback resistors"

Commit message: Updated Schematics
Added:
- digital pot
- digital loads
- updated  switch sheet to block two ways before battery
Changed lines of the file:
@@
 LIBS:tps7a7002
 LIBS:max5395
+LIBS:ina210
+LIBS:ncs20071
 LIBS:EPS-cache
 EELAYER 25 0
@@
 $Descr A4 11693 8268
 encoding utf-8
-Sheet 6 13
+Sheet 6 14
 Title "Boost converters"
 Date "2018-02-13"
@@
 	3075 1800 3075 1850
 Wire Wire Line
-	2650 1850 3075 1850
-Wire Wire Line
-	3075 1850 3275 1850
+	2650 1850 3275 1850
 Wire Wire Line
 	2650 1450 3075 1450
 Wire Wire Line
-	3075 1400 3075 1450
-Wire Wire Line
-	3075 1450 3075 1500
+	3075 1400 3075 1500
 Connection ~ 3075 1450
 $Comp
@@
 $EndComp
 Wire Wire Line
-	3075 875  3075 925
-Wire Wire Line
-	3075 925  3075 1000
+	3075 875  3075 1000
 Wire Wire Line
 	3075 600  3075 675
 Wire Wire Line
-	2175 600  2700 600
-Wire Wire Line
-	2700 600  3075 600
+	2175 600  3075 600
 $Comp
 L GND #PWR?
@@
 $EndComp
 Wire Wire Line
-	2650 2100 3450 2100
-Wire Wire Line
-	3450 2100 4200 2100
-Wire Wire Line
-	4200 2100 4675 2100
+	2650 2100 4675 2100
 Wire Wire Line
 	4200 2050 4200 2100
@@
 FB1
 Wire Wire Line
-	3900 925  4200 925
-Wire Wire Line
-	4200 925  4650 925
-Wire Wire Line
-	4650 925  4925 925
-Wire Wire Line
-	4925 925  5225 925
+	3900 925  5225 925
 Wire Wire Line
 	4200 925  4200 1750
@@
 Vcc1
 Wire Wire Line
-	1075 1750 1300 1750
-Wire Wire Line
-	1300 1750 1500 1750
+	1075 1750 1500 1750
 Text GLabel 4925 825  1    60   Output ~ 0
 Vcc1
 Wire Wire Line
-	4925 825  4925 925
-Wire Wire Line
-	4925 925  4925 975
+	4925 825  4925 975
 Connection ~ 4925 925
 Wire Wire Line
@@
 	950  2500 750  2500
 Wire Wire Line
-	750  2500 750  2575
-Wire Wire Line
-	750  2575 750  2650
+	750  2500 750  2650
 Wire Wire Line
 	750  2650 950  2650
@@
 	3075 4200 3075 4250
 Wire Wire Line
-	2650 4250 3075 4250
-Wire Wire Line
-	3075 4250 3275 4250
+	2650 4250 3275 4250
 Wire Wire Line
 	2650 3850 3075 3850
 Wire Wire Line
-	3075 3800 3075 3850
-Wire Wire Line
-	3075 3850 3075 3900
+	3075 3800 3075 3900
 Connection ~ 3075 3850
 $Comp
@@
 $EndComp
 Wire Wire Line
-	3075 3275 3075 3325
-Wire Wire Line
-	3075 3325 3075 3400
+	3075 3275 3075 3400
 Wire Wire Line
 	3075 3000 3075 3075
 Wire Wire Line
-	2175 3000 2700 3000
-Wire Wire Line
-	2700 3000 3075 3000
+	2175 3000 3075 3000
 $Comp
 L GND #PWR?
@@
 $EndComp
 Wire Wire Line
-	2650 4500 3450 4500
-Wire Wire Line
-	3450 4500 4200 4500
-Wire Wire Line
-	4200 4500 4675 4500
+	2650 4500 4675 4500
 Wire Wire Line
 	4200 4450 4200 4500
@@
 FB2
 Wire Wire Line
-	3900 3325 4200 3325
-Wire Wire Line
-	4200 3325 4650 3325
-Wire Wire Line
-	4650 3325 4925 3325
-Wire Wire Line
-	4925 3325 5225 3325
+	3900 3325 5225 3325
 Wire Wire Line
 	4200 3325 4200 4150
@@
 Vcc2
 Wire Wire Line
-	1075 4150 1300 4150
-Wire Wire Line
-	1300 4150 1500 4150
+	1075 4150 1500 4150
 Text GLabel 4925 3225 1    60   Output ~ 0
 Vcc2
 Wire Wire Line
-	4925 3225 4925 3325
-Wire Wire Line
-	4925 3325 4925 3375
+	4925 3225 4925 3375
 Connection ~ 4925 3325
 Wire Wire Line
@@
 	950  4900 750  4900
 Wire Wire Line
-	750  4900 750  4975
-Wire Wire Line
-	750  4975 750  5050
+	750  4900 750  5050
 Wire Wire Line
 	750  5050 950  5050
@@
 	3075 6600 3075 6650
 Wire Wire Line
-	2650 6650 3075 6650
-Wire Wire Line
-	3075 6650 3275 6650
+	2650 6650 3275 6650
 Wire Wire Line
 	2650 6250 3075 6250
 Wire Wire Line
-	3075 6200 3075 6250
-Wire Wire Line
-	3075 6250 3075 6300
+	3075 6200 3075 6300
 Connection ~ 3075 6250
 $Comp
@@
 $EndComp
 Wire Wire Line
-	3075 5675 3075 5725
-Wire Wire Line
-	3075 5725 3075 5800
+	3075 5675 3075 5800
 Wire Wire Line
 	3075 5400 3075 5475
 Wire Wire Line
-	2175 5400 2700 5400
-Wire Wire Line
-	2700 5400 3075 5400
+	2175 5400 3075 5400
 $Comp
 L GND #PWR?
@@
 $EndComp
 Wire Wire Line
-	2650 6900 3450 6900
-Wire Wire Line
-	3450 6900 4200 6900
-Wire Wire Line
-	4200 6900 4675 6900
+	2650 6900 4675 6900
 Wire Wire Line
 	4200 6850 4200 6900
@@
 FB3
 Wire Wire Line
-	3900 5725 4200 5725
-Wire Wire Line
-	4200 5725 4650 5725
-Wire Wire Line
-	4650 5725 4925 5725
-Wire Wire Line
-	4925 5725 5225 5725
+	3900 5725 5225 5725
 Wire Wire Line
 	4200 5725 4200 6550
@@
 Vcc3
 Wire Wire Line
-	1075 6550 1300 6550
-Wire Wire Line
-	1300 6550 1500 6550
+	1075 6550 1500 6550
 Text GLabel 4925 5625 1    60   Output ~ 0
 Vcc3
 Wire Wire Line
-	4925 5625 4925 5725
-Wire Wire Line
-	4925 5725 4925 5775
+	4925 5625 4925 5775
 Connection ~ 4925 5725
 Wire Wire Line
@@
 	950  7300 750  7300
 Wire Wire Line
-	750  7300 750  7375
-Wire Wire Line
-	750  7375 750  7450
+	750  7300 750  7450
 Wire Wire Line
 	750  7450 950  7450
