File: EPS/Battery_pack.sch (KiCad schematic (older format))
At the start: 11 parts

Commit message: Add files via upload
Parts:
- added Q?: Q_NMOS_DGS, symbol Q_NMOS_DGS
- added R?: 10k, symbol R
- added R? (x4): R, symbol R
- added Resistive_wire_connector: Molex, Connectors_Molex:Molex_KK-6410-02_02x2.54mm_Straight, symbol Conn_01x02
Connections:
- net BATT+: now also R?.1, Resistive_wire_connector.1 (Pin_1)
- net GND: now also Q?.3 (S), R?.1, R?.1, R?.2
- net at BT?.1 (+), BT?.2 (-), R?.2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: now also R?.1
- new net: Q?.1 (D), Resistive_wire_connector.2 (Pin_2)
- new net BATT_CELL1_VOLTAGE: R?.2, R?.2
- new net BATT_CELL2_VOLTAGE: R?.2, R?.2
- new net BATT_HEATER: Q?.2 (G), R?.1
Changed lines of the file:
@@
 Text Notes 925  1900 0    60   ~ 0
 Do we need over-current protection?\n(Most likely yes, but does cells already\nprovide overdischarge protection?)\n
-Wire Notes Line
-	1150 2075 1150 2275
 Text Notes 900  2400 0    60   ~ 0
 Aleksi, find out ;)
@@
 	0    1    1    0
 $EndComp
-Wire Wire Line
-	4500 4175 5150 4175
-Wire Wire Line
-	4700 4125 4700 4725
-Wire Wire Line
-	3925 4175 4200 4175
-Wire Wire Line
-	3925 4175 3925 4575
-Wire Wire Line
-	3925 4575 4200 4575
-Wire Wire Line
-	3925 4375 3525 4375
-Wire Wire Line
-	3525 4175 3525 4600
-Connection ~ 3925 4375
-Connection ~ 3525 4375
 $Comp
 L C C?
@@
 	1    0    0    -1
 $EndComp
-Connection ~ 4700 4175
 $Comp
 L R R?
@@
 	0    1    1    0
 $EndComp
-Wire Wire Line
-	4700 3825 4700 3775
-Wire Wire Line
-	4500 3775 5050 3775
-Wire Wire Line
-	4200 3775 3525 3775
-Wire Wire Line
-	3525 3450 3525 3875
-Wire Wire Line
-	5050 3775 5050 4025
-Connection ~ 4700 3775
-Wire Wire Line
-	4500 4575 5050 4575
-Wire Wire Line
-	5050 4025 5150 4025
-Wire Wire Line
-	5150 4325 5050 4325
-Wire Wire Line
-	5050 4325 5050 4575
-Wire Wire Line
-	3525 5125 3525 4900
-Wire Wire Line
-	4700 5125 4700 5025
 $Comp
 L C C?
@@
 	1    0    0    -1
 $EndComp
-Wire Wire Line
-	5150 4475 5100 4475
-Wire Wire Line
-	5100 4475 5100 4725
-Wire Wire Line
-	5100 5125 5100 5025
-Wire Wire Line
-	6300 5125 6300 4325
-Wire Wire Line
-	6300 4475 6200 4475
-Wire Wire Line
-	6300 4325 6200 4325
-Connection ~ 6300 4475
-Wire Wire Line
-	3525 3450 7075 3450
-Connection ~ 3525 3775
 $Comp
 L R R?
@@
 	1    0    0    -1
 $EndComp
-Wire Wire Line
-	6200 4175 6650 4175
-Wire Wire Line
-	6650 3850 6650 4700
-Wire Wire Line
-	6650 3550 6650 3450
-Connection ~ 6650 3450
 $Comp
 L C C?
@@
 	1    0    0    -1
 $EndComp
-Connection ~ 6650 4175
-Wire Wire Line
-	6650 5125 6650 5000
-Wire Wire Line
-	3525 5125 7075 5125
-Connection ~ 4700 5125
-Connection ~ 5100 5125
-Connection ~ 6300 5125
-Connection ~ 6650 5125
 Text HLabel 7075 5125 2    60   BiDi ~ 0
 BATT-
@@
 	1    0    0    -1
 $EndComp
+Text Notes 6500 5375 0    60   ~ 0
+HIGH => overvoltage condition\nWhat is voltage level that is outputed?
+Text Notes 3725 2850 0    60   ~ 0
+Choose resistor and capacitor values for\noptimal balancing current\n
+Text Notes 2350 3700 0    60   ~ 0
+Battery voltage\nand current \nmeasurements here
+$Comp
+L Conn_01x02 Resistive_wire_connector
+U 1 1 5A8DA99C
+P 7400 3800
+F 0 "Resistive_wire_connector" H 7400 3900 50  0000 C CNN
+F 1 "Molex" H 7400 3600 50  0000 C CNN
+F 2 "Connectors_Molex:Molex_KK-6410-02_02x2.54mm_Straight" H 7400 3800 50  0001 C CNN
+F 3 "" H 7400 3800 50  0001 C CNN
+	1    7400 3800
+	1    0    0    -1
+$EndComp
+$Comp
+L Q_NMOS_DGS Q?
+U 1 1 5A8DAAA5
+P 7050 4400
+F 0 "Q?" H 6850 4450 50  0000 L CNN
+F 1 "Q_NMOS_DGS" H 6550 4550 50  0000 L CNN
+F 2 "" H 7250 4500 50  0001 C CNN
+F 3 "" H 7050 4400 50  0001 C CNN
+	1    7050 4400
+	-1   0    0    -1
+$EndComp
+$Comp
+L R R?
+U 1 1 5A8DAE10
+P 7250 4700
+F 0 "R?" V 7330 4700 50  0000 C CNN
+F 1 "10k" V 7250 4700 50  0000 C CNN
+F 2 "" V 7180 4700 50  0001 C CNN
+F 3 "" H 7250 4700 50  0001 C CNN
+	1    7250 4700
+	1    0    0    -1
+$EndComp
+$Comp
+L GND #PWR?
+U 1 1 5A8DAE81
+P 7250 4850
+F 0 "#PWR?" H 7250 4600 50  0001 C CNN
+F 1 "GND" H 7250 4700 50  0000 C CNN
+F 2 "" H 7250 4850 50  0001 C CNN
+F 3 "" H 7250 4850 50  0001 C CNN
+	1    7250 4850
+	1    0    0    -1
+$EndComp
+Text HLabel 7625 4400 2    60   Input ~ 0
+BATT_HEATER
+$Comp
+L R R?
+U 1 1 5A8EC8AE
+P 3025 3775
+F 0 "R?" V 3105 3775 50  0000 C CNN
+F 1 "R" V 3025 3775 50  0000 C CNN
+F 2 "" V 2955 3775 50  0001 C CNN
+F 3 "" H 3025 3775 50  0001 C CNN
+	1    3025 3775
+	0    1    1    0
+$EndComp
+$Comp
+L R R?
+U 1 1 5A8EC9BC
+P 3025 4375
+F 0 "R?" V 3105 4375 50  0000 C CNN
+F 1 "R" V 3025 4375 50  0000 C CNN
+F 2 "" V 2955 4375 50  0001 C CNN
+F 3 "" H 3025 4375 50  0001 C CNN
+	1    3025 4375
+	0    1    1    0
+$EndComp
+$Comp
+L R R?
+U 1 1 5A8ECC34
+P 2875 4025
+F 0 "R?" V 2955 4025 50  0000 C CNN
+F 1 "R" V 2875 4025 50  0000 C CNN
+F 2 "" V 2805 4025 50  0001 C CNN
+F 3 "" H 2875 4025 50  0001 C CNN
+	1    2875 4025
+	-1   0    0    1
+$EndComp
+$Comp
+L R R?
+U 1 1 5A8ECCC7
+P 2875 4650
+F 0 "R?" V 2955 4650 50  0000 C CNN
+F 1 "R" V 2875 4650 50  0000 C CNN
+F 2 "" V 2805 4650 50  0001 C CNN
+F 3 "" H 2875 4650 50  0001 C CNN
+	1    2875 4650
+	-1   0    0    1
+$EndComp
+$Comp
+L GND #PWR?
+U 1 1 5A8ECDA3
+P 2875 4175
+F 0 "#PWR?" H 2875 3925 50  0001 C CNN
+F 1 "GND" H 3000 4125 50  0000 C CNN
+F 2 "" H 2875 4175 50  0001 C CNN
+F 3 "" H 2875 4175 50  0001 C CNN
+	1    2875 4175
+	1    0    0    -1
+$EndComp
+$Comp
+L GND #PWR?
+U 1 1 5A8ECDEB
+P 2875 4800
+F 0 "#PWR?" H 2875 4550 50  0001 C CNN
+F 1 "GND" H 2875 4650 50  0000 C CNN
+F 2 "" H 2875 4800 50  0001 C CNN
+F 3 "" H 2875 4800 50  0001 C CNN
+	1    2875 4800
+	1    0    0    -1
+$EndComp
+Wire Notes Line
+	1150 2075 1150 2275
+Wire Wire Line
+	4500 4175 5150 4175
+Wire Wire Line
+	4700 4125 4700 4725
+Wire Wire Line
+	3925 4175 4200 4175
+Wire Wire Line
+	3925 4175 3925 4575
+Wire Wire Line
+	3925 4575 4200 4575
+Wire Wire Line
+	3175 4375 3925 4375
+Wire Wire Line
+	3525 4175 3525 4600
+Connection ~ 3925 4375
+Connection ~ 3525 4375
+Connection ~ 4700 4175
+Wire Wire Line
+	4700 3825 4700 3775
+Wire Wire Line
+	4500 3775 5050 3775
+Wire Wire Line
+	3175 3775 4200 3775
+Wire Wire Line
+	3525 3450 3525 3875
+Wire Wire Line
+	5050 3775 5050 4025
+Connection ~ 4700 3775
+Wire Wire Line
+	4500 4575 5050 4575
+Wire Wire Line
+	5050 4025 5150 4025
+Wire Wire Line
+	5150 4325 5050 4325
+Wire Wire Line
+	5050 4325 5050 4575
+Wire Wire Line
+	3525 5125 3525 4900
+Wire Wire Line
+	4700 5125 4700 5025
+Wire Wire Line
+	5150 4475 5100 4475
+Wire Wire Line
+	5100 4475 5100 4725
+Wire Wire Line
+	5100 5125 5100 5025
+Wire Wire Line
+	6300 5125 6300 4325
+Wire Wire Line
+	6300 4475 6200 4475
+Wire Wire Line
+	6300 4325 6200 4325
+Connection ~ 6300 4475
+Wire Wire Line
+	3525 3450 7075 3450
+Connection ~ 3525 3775
+Wire Wire Line
+	6200 4175 6650 4175
+Wire Wire Line
+	6650 3850 6650 4700
+Wire Wire Line
+	6650 3550 6650 3450
+Connection ~ 6650 3450
+Connection ~ 6650 4175
+Wire Wire Line
+	6650 5125 6650 5000
+Wire Wire Line
+	3525 5125 7075 5125
+Connection ~ 4700 5125
+Connection ~ 5100 5125
+Connection ~ 6300 5125
+Connection ~ 6650 5125
 Wire Wire Line
 	5700 5250 5700 5125
 Connection ~ 5700 5125
 Wire Notes Line
-	6350 4025 7000 4025
-Text Notes 7075 4050 0    60   ~ 0
-HIGH => overvoltage condition\nWhat is voltage level that is outputed?
-Wire Notes Line
 	4350 3650 4350 2925
-Text Notes 3725 2850 0    60   ~ 0
-Choose resistor and capacitor values for\noptimal balancing current\n
 Wire Notes Line
 	4950 2925 4950 4875
@@
 Wire Notes Line
 	2700 3400 3275 3400
-Text Notes 2350 3700 0    60   ~ 0
-Battery voltage\nand current \nmeasurements here
 Wire Notes Line
 	3275 3400 3275 5175
+Wire Notes Line
+	6400 4025 6400 5300
+Wire Notes Line
+	6400 5300 6450 5300
+Wire Wire Line
+	6950 3450 6950 3800
+Wire Wire Line
+	6950 3800 7200 3800
+Connection ~ 6950 3450
+Wire Wire Line
+	7200 3900 6950 3900
+Wire Wire Line
+	6950 3900 6950 4200
+Wire Wire Line
+	6950 4600 6950 5125
+Connection ~ 6950 5125
+Wire Wire Line
+	7250 4400 7250 4550
+Wire Wire Line
+	7250 4400 7625 4400
+Wire Wire Line
+	2875 3775 2875 3875
+Wire Wire Line
+	2875 4375 2875 4500
+Wire Wire Line
+	2875 3775 2700 3775
+Wire Wire Line
+	2875 4375 2700 4375
+Text HLabel 2700 4375 0    60   Output ~ 0
+BATT_CELL1_VOLTAGE
+Text HLabel 2700 3775 0    60   Output ~ 0
+BATT_CELL2_VOLTAGE
 $EndSCHEMATC
