File: EPS/CAN_transceivers.sch (KiCad schematic (older format))
At the start: 6 parts, among them U2 SN65HVD232, U3 SN65HVD232

Commit message: Finalized SCH (beta version) and started pcb
Capacitor banks might need to be reassigned to other locations.
No RBF pin on this SCH or PCB.
Battery gound deployment switch is fully mechanical (no mosfet switch on low side).
PCB of the prototype started. Main power converters and current measuring devices layed out.
SCH still requires ESD protection diodes!
Connections:
- net CAN2_H is gone; now on net CAN_H: R4.1, U3.7 (CANH)
- net CAN2_L is gone; now on net CAN_L: R4.2, U3.6 (CANL)
- net CAN1_H renamed CAN_H
- net CAN1_L renamed CAN_L
Changed lines of the file:
@@
 	4925 2700 5025 2700
 Text HLabel 6225 2700 2    60   BiDi ~ 0
-CAN1_H
+CAN_H
 Text HLabel 6225 2800 2    60   BiDi ~ 0
-CAN1_L
+CAN_L
 Wire Wire Line
 	5825 2700 6225 2700
@@
 	4950 4500 5050 4500
 Text HLabel 6250 4500 2    60   BiDi ~ 0
-CAN2_H
+CAN_H
 Text HLabel 6250 4600 2    60   BiDi ~ 0
-CAN2_L
+CAN_L
 Wire Wire Line
 	5850 4500 6250 4500
