File: EPS/Output_telemetria.sch (KiCad schematic (older format))
At the start: 12 parts

Commit message: Updated Schematics
Added:
- digital pot
- digital loads
- updated  switch sheet to block two ways before battery
Parts:
- removed INA? (x3): INA139, symbol INA139
- added INA? (x3): INA210, symbol INA210
Connections:
- net +3V3: now also INA?.3 (V+), INA?.3 (V+), INA?.3 (V+)
- net GND: now also INA?.1 (REF), INA?.1 (REF), INA?.1 (REF), INA?.2 (GND), INA?.2 (GND), INA?.2 (GND)
- net I1_OUT: now also INA?.6 (OUT)
- net I2_OUT: now also INA?.6 (OUT)
- net I3_OUT: now also INA?.6 (OUT)
- net INA1_OUT+: now also INA?.4 (IN+)
- net INA1_OUT-: now also INA?.5 (IN-)
- net INA2_OUT+: now also INA?.4 (IN+)
- net INA2_OUT-: now also INA?.5 (IN-)
- net INA3_OUT+: now also INA?.4 (IN+)
- net INA3_OUT-: now also INA?.5 (IN-)
Changed lines of the file:
@@
 LIBS:tps7a7002
 LIBS:max5395
+LIBS:ina210
+LIBS:ncs20071
 LIBS:EPS-cache
 EELAYER 25 0
@@
 $Descr A4 11693 8268
 encoding utf-8
-Sheet 7 13
+Sheet 7 14
 Title "Output telemetria"
 Date "2018-02-12"
@@
 Comment4 ""
 $EndDescr
-$Comp
-L INA139 INA?
-U 1 1 5A824969
-P 5850 1725
-F 0 "INA?" H 5850 1450 60  0000 C CNN
-F 1 "INA139" H 5850 2000 60  0000 C CNN
-F 2 "" H 5725 1775 60  0001 C CNN
-F 3 "" H 5725 1775 60  0001 C CNN
-	1    5850 1725
-	1    0    0    -1
-$EndComp
 $Comp
 L R R_s?
@@
 Connection ~ 6400 2375
 $Comp
-L INA139 INA?
-U 1 1 5A8249B1
-P 5775 3450
-F 0 "INA?" H 5775 3175 60  0000 C CNN
-F 1 "INA139" H 5775 3725 60  0000 C CNN
-F 2 "" H 5650 3500 60  0001 C CNN
-F 3 "" H 5650 3500 60  0001 C CNN
-	1    5775 3450
-	1    0    0    -1
-$EndComp
-$Comp
 L R R_s?
 U 1 1 5A8249B8
@@
 INA2_OUT-
 Connection ~ 6325 4100
-$Comp
-L INA139 INA?
-U 1 1 5A8249F9
-P 5700 5125
-F 0 "INA?" H 5700 4850 60  0000 C CNN
-F 1 "INA139" H 5700 5400 60  0000 C CNN
-F 2 "" H 5575 5175 60  0001 C CNN
-F 3 "" H 5575 5175 60  0001 C CNN
-	1    5700 5125
-	1    0    0    -1
-$EndComp
 $Comp
 L R R_s?
@@
 Text Notes 7350 3500 0    60   ~ 0
 Need values for shunt and load resistors\n
+$Comp
+L INA210 INA?
+U 1 1 5A8C7168
+P 5575 1500
+F 0 "INA?" H 5775 1725 60  0000 C CNN
+F 1 "INA210" H 5775 1625 60  0000 C CNN
+F 2 "" H 5775 1625 60  0001 C CNN
+F 3 "" H 5775 1625 60  0001 C CNN
+	1    5575 1500
+	1    0    0    -1
+$EndComp
+$Comp
+L INA210 INA?
+U 1 1 5A8C730D
+P 5500 3225
+F 0 "INA?" H 5700 3450 60  0000 C CNN
+F 1 "INA210" H 5700 3350 60  0000 C CNN
+F 2 "" H 5700 3350 60  0001 C CNN
+F 3 "" H 5700 3350 60  0001 C CNN
+	1    5500 3225
+	1    0    0    -1
+$EndComp
+$Comp
+L INA210 INA?
+U 1 1 5A8C73D5
+P 5425 4900
+F 0 "INA?" H 5625 5125 60  0000 C CNN
+F 1 "INA210" H 5625 5025 60  0000 C CNN
+F 2 "" H 5625 5025 60  0001 C CNN
+F 3 "" H 5625 5025 60  0001 C CNN
+	1    5425 4900
+	1    0    0    -1
+$EndComp
+$Comp
+L GND #PWR?
+U 1 1 5A8C741F
+P 6150 5125
+F 0 "#PWR?" H 6150 4875 50  0001 C CNN
+F 1 "GND" H 6150 4975 50  0000 C CNN
+F 2 "" H 6150 5125 50  0001 C CNN
+F 3 "" H 6150 5125 50  0001 C CNN
+	1    6150 5125
+	0    -1   -1   0
+$EndComp
+$Comp
+L GND #PWR?
+U 1 1 5A8C747E
+P 6225 3450
+F 0 "#PWR?" H 6225 3200 50  0001 C CNN
+F 1 "GND" H 6225 3300 50  0000 C CNN
+F 2 "" H 6225 3450 50  0001 C CNN
+F 3 "" H 6225 3450 50  0001 C CNN
+	1    6225 3450
+	0    -1   -1   0
+$EndComp
+$Comp
+L GND #PWR?
+U 1 1 5A8C753D
+P 6300 1725
+F 0 "#PWR?" H 6300 1475 50  0001 C CNN
+F 1 "GND" H 6300 1575 50  0000 C CNN
+F 2 "" H 6300 1725 50  0001 C CNN
+F 3 "" H 6300 1725 50  0001 C CNN
+	1    6300 1725
+	0    -1   -1   0
+$EndComp
 $EndSCHEMATC

Commit message: Finalized SCH (beta version) and started pcb
Capacitor banks might need to be reassigned to other locations.
No RBF pin on this SCH or PCB.
Battery gound deployment switch is fully mechanical (no mosfet switch on low side).
PCB of the prototype started. Main power converters and current measuring devices layed out.
SCH still requires ESD protection diodes!
Parts:
- removed R_l? (x3): R, symbol R
- C44, C45, C46: renamed from C?; footprint (none) -> Capacitors_SMD:C_0603
- INA4, INA5, INA6: renamed from INA?; footprint (none) -> TO_SOT_Packages_SMD:SOT-363_SC-70-6
- R_s4, R_s5, R_s6: renamed from R_s?; footprint (none) -> Resistors_SMD:R_0805
Changed lines of the file:
@@
 Sheet 7 14
 Title "Output telemetria"
-Date "2018-02-12"
+Date "2018-02-22"
 Rev "R1"
 Comp ""
@@
 $EndDescr
 $Comp
-L R R_s?
+L R R_s6
 U 1 1 5A824970
 P 5850 2375
-F 0 "R_s?" V 5930 2375 50  0000 C CNN
+F 0 "R_s6" V 5930 2375 50  0000 C CNN
 F 1 "R" V 5850 2375 50  0000 C CNN
-F 2 "" V 5780 2375 50  0001 C CNN
+F 2 "Resistors_SMD:R_0805" V 5780 2375 50  0001 C CNN
 F 3 "" H 5850 2375 50  0001 C CNN
 	1    5850 2375
@@
 $EndComp
 $Comp
-L R R_l?
-U 1 1 5A824977
-P 4525 1800
-F 0 "R_l?" V 4605 1800 50  0000 C CNN
-F 1 "R" V 4525 1800 50  0000 C CNN
-F 2 "" V 4455 1800 50  0001 C CNN
-F 3 "" H 4525 1800 50  0001 C CNN
-	1    4525 1800
-	1    0    0    -1
-$EndComp
-$Comp
-L C C?
+L C C46
 U 1 1 5A82497E
 P 6625 1375
-F 0 "C?" H 6650 1475 50  0000 L CNN
+F 0 "C46" H 6650 1475 50  0000 L CNN
 F 1 "0.1u" H 6650 1275 50  0000 L CNN
-F 2 "" H 6663 1225 50  0001 C CNN
+F 2 "Capacitors_SMD:C_0603" H 6663 1225 50  0001 C CNN
 F 3 "" H 6625 1375 50  0001 C CNN
 	1    6625 1375
@@
 $EndComp
 $Comp
-L GND #PWR?
+L GND #PWR085
 U 1 1 5A824985
 P 5025 1725
-F 0 "#PWR?" H 5025 1475 50  0001 C CNN
+F 0 "#PWR085" H 5025 1475 50  0001 C CNN
 F 1 "GND" H 5025 1575 50  0000 C CNN
 F 2 "" H 5025 1725 50  0001 C CNN
@@
 $EndComp
 $Comp
-L +3.3V #PWR?
+L +3.3V #PWR086
 U 1 1 5A82498B
 P 6475 1025
-F 0 "#PWR?" H 6475 875 50  0001 C CNN
+F 0 "#PWR086" H 6475 875 50  0001 C CNN
 F 1 "+3.3V" H 6475 1165 50  0000 C CNN
 F 2 "" H 6475 1025 50  0001 C CNN
@@
 Connection ~ 6475 1375
 $Comp
-L GND #PWR?
+L GND #PWR087
 U 1 1 5A824994
 P 7000 1375
-F 0 "#PWR?" H 7000 1125 50  0001 C CNN
+F 0 "#PWR087" H 7000 1125 50  0001 C CNN
 F 1 "GND" H 7000 1225 50  0000 C CNN
 F 2 "" H 7000 1375 50  0001 C CNN
@@
 Wire Wire Line
 	6400 1875 6300 1875
-$Comp
-L GND #PWR?
-U 1 1 5A8249A2
-P 4525 2050
-F 0 "#PWR?" H 4525 1800 50  0001 C CNN
-F 1 "GND" H 4525 1900 50  0000 C CNN
-F 2 "" H 4525 2050 50  0001 C CNN
-F 3 "" H 4525 2050 50  0001 C CNN
-	1    4525 2050
-	1    0    0    -1
-$EndComp
-Wire Wire Line
-	4525 2050 4525 1950
 Wire Wire Line
 	4400 1575 5375 1575
-Wire Wire Line
-	4525 1575 4525 1650
 Text HLabel 4400 1575 0    60   Output ~ 0
 I1_OUT
-Connection ~ 4525 1575
 Text HLabel 5150 2375 0    60   Input ~ 0
 INA1_OUT+
@@
 Connection ~ 6400 2375
 $Comp
-L R R_s?
+L R R_s5
 U 1 1 5A8249B8
 P 5775 4100
-F 0 "R_s?" V 5855 4100 50  0000 C CNN
+F 0 "R_s5" V 5855 4100 50  0000 C CNN
 F 1 "R" V 5775 4100 50  0000 C CNN
-F 2 "" V 5705 4100 50  0001 C CNN
+F 2 "Resistors_SMD:R_0805" V 5705 4100 50  0001 C CNN
 F 3 "" H 5775 4100 50  0001 C CNN
 	1    5775 4100
@@
 $EndComp
 $Comp
-L R R_l?
-U 1 1 5A8249BF
-P 4450 3525
-F 0 "R_l?" V 4530 3525 50  0000 C CNN
-F 1 "R" V 4450 3525 50  0000 C CNN
-F 2 "" V 4380 3525 50  0001 C CNN
-F 3 "" H 4450 3525 50  0001 C CNN
-	1    4450 3525
-	1    0    0    -1
-$EndComp
-$Comp
-L C C?
+L C C45
 U 1 1 5A8249C6
 P 6550 3100
-F 0 "C?" H 6575 3200 50  0000 L CNN
+F 0 "C45" H 6575 3200 50  0000 L CNN
 F 1 "0.1u" H 6575 3000 50  0000 L CNN
-F 2 "" H 6588 2950 50  0001 C CNN
+F 2 "Capacitors_SMD:C_0603" H 6588 2950 50  0001 C CNN
 F 3 "" H 6550 3100 50  0001 C CNN
 	1    6550 3100
@@
 $EndComp
 $Comp
-L GND #PWR?
+L GND #PWR088
 U 1 1 5A8249CD
 P 4950 3450
-F 0 "#PWR?" H 4950 3200 50  0001 C CNN
+F 0 "#PWR088" H 4950 3200 50  0001 C CNN
 F 1 "GND" H 4950 3300 50  0000 C CNN
 F 2 "" H 4950 3450 50  0001 C CNN
@@
 $EndComp
 $Comp
-L +3.3V #PWR?
+L +3.3V #PWR089
 U 1 1 5A8249D3
 P 6400 2750
-F 0 "#PWR?" H 6400 2600 50  0001 C CNN
+F 0 "#PWR089" H 6400 2600 50  0001 C CNN
 F 1 "+3.3V" H 6400 2890 50  0000 C CNN
 F 2 "" H 6400 2750 50  0001 C CNN
@@
 Connection ~ 6400 3100
 $Comp
-L GND #PWR?
+L GND #PWR090
 U 1 1 5A8249DC
 P 6925 3100
-F 0 "#PWR?" H 6925 2850 50  0001 C CNN
+F 0 "#PWR090" H 6925 2850 50  0001 C CNN
 F 1 "GND" H 6925 2950 50  0000 C CNN
 F 2 "" H 6925 3100 50  0001 C CNN
@@
 Wire Wire Line
 	6325 3600 6225 3600
-$Comp
-L GND #PWR?
-U 1 1 5A8249EA
-P 4450 3775
-F 0 "#PWR?" H 4450 3525 50  0001 C CNN
-F 1 "GND" H 4450 3625 50  0000 C CNN
-F 2 "" H 4450 3775 50  0001 C CNN
-F 3 "" H 4450 3775 50  0001 C CNN
-	1    4450 3775
-	1    0    0    -1
-$EndComp
-Wire Wire Line
-	4450 3775 4450 3675
 Wire Wire Line
 	4325 3300 5300 3300
-Wire Wire Line
-	4450 3300 4450 3375
 Text HLabel 4325 3300 0    60   Output ~ 0
 I2_OUT
-Connection ~ 4450 3300
 Text HLabel 5075 4100 0    60   Input ~ 0
 INA2_OUT+
@@
 Connection ~ 6325 4100
 $Comp
-L R R_s?
+L R R_s4
 U 1 1 5A824A00
 P 5700 5775
-F 0 "R_s?" V 5780 5775 50  0000 C CNN
+F 0 "R_s4" V 5780 5775 50  0000 C CNN
 F 1 "R" V 5700 5775 50  0000 C CNN
-F 2 "" V 5630 5775 50  0001 C CNN
+F 2 "Resistors_SMD:R_0805" V 5630 5775 50  0001 C CNN
 F 3 "" H 5700 5775 50  0001 C CNN
 	1    5700 5775
@@
 $EndComp
 $Comp
-L R R_l?
-U 1 1 5A824A07
-P 4375 5200
-F 0 "R_l?" V 4455 5200 50  0000 C CNN
-F 1 "R" V 4375 5200 50  0000 C CNN
-F 2 "" V 4305 5200 50  0001 C CNN
-F 3 "" H 4375 5200 50  0001 C CNN
-	1    4375 5200
-	1    0    0    -1
-$EndComp
-$Comp
-L C C?
+L C C44
 U 1 1 5A824A0E
 P 6475 4775
-F 0 "C?" H 6500 4875 50  0000 L CNN
+F 0 "C44" H 6500 4875 50  0000 L CNN
 F 1 "0.1u" H 6500 4675 50  0000 L CNN
-F 2 "" H 6513 4625 50  0001 C CNN
+F 2 "Capacitors_SMD:C_0603" H 6513 4625 50  0001 C CNN
 F 3 "" H 6475 4775 50  0001 C CNN
 	1    6475 4775
@@
 $EndComp
 $Comp
-L GND #PWR?
+L GND #PWR091
 U 1 1 5A824A15
 P 4875 5125
-F 0 "#PWR?" H 4875 4875 50  0001 C CNN
+F 0 "#PWR091" H 4875 4875 50  0001 C CNN
 F 1 "GND" H 4875 4975 50  0000 C CNN
 F 2 "" H 4875 5125 50  0001 C CNN
@@
 $EndComp
 $Comp
-L +3.3V #PWR?
+L +3.3V #PWR092
 U 1 1 5A824A1B
 P 6325 4425
-F 0 "#PWR?" H 6325 4275 50  0001 C CNN
+F 0 "#PWR092" H 6325 4275 50  0001 C CNN
 F 1 "+3.3V" H 6325 4565 50  0000 C CNN
 F 2 "" H 6325 4425 50  0001 C CNN
@@
 Connection ~ 6325 4775
 $Comp
-L GND #PWR?
+L GND #PWR093
 U 1 1 5A824A24
 P 6850 4775
-F 0 "#PWR?" H 6850 4525 50  0001 C CNN
+F 0 "#PWR093" H 6850 4525 50  0001 C CNN
 F 1 "GND" H 6850 4625 50  0000 C CNN
 F 2 "" H 6850 4775 50  0001 C CNN
@@
 Wire Wire Line
 	6250 5275 6150 5275
-$Comp
-L GND #PWR?
-U 1 1 5A824A32
-P 4375 5450
-F 0 "#PWR?" H 4375 5200 50  0001 C CNN
-F 1 "GND" H 4375 5300 50  0000 C CNN
-F 2 "" H 4375 5450 50  0001 C CNN
-F 3 "" H 4375 5450 50  0001 C CNN
-	1    4375 5450
-	1    0    0    -1
-$EndComp
-Wire Wire Line
-	4375 5450 4375 5350
 Wire Wire Line
 	4250 4975 5225 4975
-Wire Wire Line
-	4375 4975 4375 5050
 Text HLabel 4250 4975 0    60   Output ~ 0
 I3_OUT
-Connection ~ 4375 4975
 Text HLabel 5000 5775 0    60   Input ~ 0
 INA3_OUT+
@@
 Need values for shunt and load resistors\n
 $Comp
-L INA210 INA?
+L INA210 INA6
 U 1 1 5A8C7168
 P 5575 1500
-F 0 "INA?" H 5775 1725 60  0000 C CNN
+F 0 "INA6" H 5775 1725 60  0000 C CNN
 F 1 "INA210" H 5775 1625 60  0000 C CNN
-F 2 "" H 5775 1625 60  0001 C CNN
+F 2 "TO_SOT_Packages_SMD:SOT-363_SC-70-6" H 5775 1625 60  0001 C CNN
 F 3 "" H 5775 1625 60  0001 C CNN
 	1    5575 1500
@@
 $EndComp
 $Comp
-L INA210 INA?
+L INA210 INA5
 U 1 1 5A8C730D
 P 5500 3225
-F 0 "INA?" H 5700 3450 60  0000 C CNN
+F 0 "INA5" H 5700 3450 60  0000 C CNN
 F 1 "INA210" H 5700 3350 60  0000 C CNN
-F 2 "" H 5700 3350 60  0001 C CNN
+F 2 "TO_SOT_Packages_SMD:SOT-363_SC-70-6" H 5700 3350 60  0001 C CNN
 F 3 "" H 5700 3350 60  0001 C CNN
 	1    5500 3225
@@
 $EndComp
 $Comp
-L INA210 INA?
+L INA210 INA4
 U 1 1 5A8C73D5
 P 5425 4900
-F 0 "INA?" H 5625 5125 60  0000 C CNN
+F 0 "INA4" H 5625 5125 60  0000 C CNN
 F 1 "INA210" H 5625 5025 60  0000 C CNN
-F 2 "" H 5625 5025 60  0001 C CNN
+F 2 "TO_SOT_Packages_SMD:SOT-363_SC-70-6" H 5625 5025 60  0001 C CNN
 F 3 "" H 5625 5025 60  0001 C CNN
 	1    5425 4900
@@
 $EndComp
 $Comp
-L GND #PWR?
+L GND #PWR094
 U 1 1 5A8C741F
 P 6150 5125
-F 0 "#PWR?" H 6150 4875 50  0001 C CNN
+F 0 "#PWR094" H 6150 4875 50  0001 C CNN
 F 1 "GND" H 6150 4975 50  0000 C CNN
 F 2 "" H 6150 5125 50  0001 C CNN
@@
 $EndComp
 $Comp
-L GND #PWR?
+L GND #PWR095
 U 1 1 5A8C747E
 P 6225 3450
-F 0 "#PWR?" H 6225 3200 50  0001 C CNN
+F 0 "#PWR095" H 6225 3200 50  0001 C CNN
 F 1 "GND" H 6225 3300 50  0000 C CNN
 F 2 "" H 6225 3450 50  0001 C CNN
@@
 $EndComp
 $Comp
-L GND #PWR?
+L GND #PWR096
 U 1 1 5A8C753D
 P 6300 1725
-F 0 "#PWR?" H 6300 1475 50  0001 C CNN
+F 0 "#PWR096" H 6300 1475 50  0001 C CNN
 F 1 "GND" H 6300 1575 50  0000 C CNN
 F 2 "" H 6300 1725 50  0001 C CNN

Commit message: PCB updated
Added testpoints and updated PCB
Parts:
- added TP13, TP14, TP15: TEST, Measurement_Points:Measurement_Point_Round-SMD-Pad_Small, symbol TEST
Connections:
- net I1_OUT: now also TP13.1
- net I2_OUT: now also TP14.1
- net I3_OUT: now also TP15.1
Changed lines of the file:
@@
 $EndComp
 $Comp
-L GND #PWR085
+L GND #PWR084
 U 1 1 5A824985
 P 5025 1725
-F 0 "#PWR085" H 5025 1475 50  0001 C CNN
+F 0 "#PWR084" H 5025 1475 50  0001 C CNN
 F 1 "GND" H 5025 1575 50  0000 C CNN
 F 2 "" H 5025 1725 50  0001 C CNN
@@
 $EndComp
 $Comp
-L +3.3V #PWR086
+L +3.3V #PWR085
 U 1 1 5A82498B
 P 6475 1025
-F 0 "#PWR086" H 6475 875 50  0001 C CNN
+F 0 "#PWR085" H 6475 875 50  0001 C CNN
 F 1 "+3.3V" H 6475 1165 50  0000 C CNN
 F 2 "" H 6475 1025 50  0001 C CNN
@@
 Connection ~ 6475 1375
 $Comp
-L GND #PWR087
+L GND #PWR086
 U 1 1 5A824994
 P 7000 1375
-F 0 "#PWR087" H 7000 1125 50  0001 C CNN
+F 0 "#PWR086" H 7000 1125 50  0001 C CNN
 F 1 "GND" H 7000 1225 50  0000 C CNN
 F 2 "" H 7000 1375 50  0001 C CNN
@@
 $EndComp
 $Comp
-L GND #PWR088
+L GND #PWR087
 U 1 1 5A8249CD
 P 4950 3450
-F 0 "#PWR088" H 4950 3200 50  0001 C CNN
+F 0 "#PWR087" H 4950 3200 50  0001 C CNN
 F 1 "GND" H 4950 3300 50  0000 C CNN
 F 2 "" H 4950 3450 50  0001 C CNN
@@
 $EndComp
 $Comp
-L +3.3V #PWR089
+L +3.3V #PWR088
 U 1 1 5A8249D3
 P 6400 2750
-F 0 "#PWR089" H 6400 2600 50  0001 C CNN
+F 0 "#PWR088" H 6400 2600 50  0001 C CNN
 F 1 "+3.3V" H 6400 2890 50  0000 C CNN
 F 2 "" H 6400 2750 50  0001 C CNN
@@
 Connection ~ 6400 3100
 $Comp
-L GND #PWR090
+L GND #PWR089
 U 1 1 5A8249DC
 P 6925 3100
-F 0 "#PWR090" H 6925 2850 50  0001 C CNN
+F 0 "#PWR089" H 6925 2850 50  0001 C CNN
 F 1 "GND" H 6925 2950 50  0000 C CNN
 F 2 "" H 6925 3100 50  0001 C CNN
@@
 $EndComp
 $Comp
-L GND #PWR091
+L GND #PWR090
 U 1 1 5A824A15
 P 4875 5125
-F 0 "#PWR091" H 4875 4875 50  0001 C CNN
+F 0 "#PWR090" H 4875 4875 50  0001 C CNN
 F 1 "GND" H 4875 4975 50  0000 C CNN
 F 2 "" H 4875 5125 50  0001 C CNN
@@
 $EndComp
 $Comp
-L +3.3V #PWR092
+L +3.3V #PWR091
 U 1 1 5A824A1B
 P 6325 4425
-F 0 "#PWR092" H 6325 4275 50  0001 C CNN
+F 0 "#PWR091" H 6325 4275 50  0001 C CNN
 F 1 "+3.3V" H 6325 4565 50  0000 C CNN
 F 2 "" H 6325 4425 50  0001 C CNN
@@
 Connection ~ 6325 4775
 $Comp
-L GND #PWR093
+L GND #PWR092
 U 1 1 5A824A24
 P 6850 4775
-F 0 "#PWR093" H 6850 4525 50  0001 C CNN
+F 0 "#PWR092" H 6850 4525 50  0001 C CNN
 F 1 "GND" H 6850 4625 50  0000 C CNN
 F 2 "" H 6850 4775 50  0001 C CNN
@@
 $EndComp
 $Comp
-L GND #PWR094
+L GND #PWR093
 U 1 1 5A8C741F
 P 6150 5125
-F 0 "#PWR094" H 6150 4875 50  0001 C CNN
+F 0 "#PWR093" H 6150 4875 50  0001 C CNN
 F 1 "GND" H 6150 4975 50  0000 C CNN
 F 2 "" H 6150 5125 50  0001 C CNN
@@
 $EndComp
 $Comp
-L GND #PWR095
+L GND #PWR094
 U 1 1 5A8C747E
 P 6225 3450
-F 0 "#PWR095" H 6225 3200 50  0001 C CNN
+F 0 "#PWR094" H 6225 3200 50  0001 C CNN
 F 1 "GND" H 6225 3300 50  0000 C CNN
 F 2 "" H 6225 3450 50  0001 C CNN
@@
 $EndComp
 $Comp
-L GND #PWR096
+L GND #PWR095
 U 1 1 5A8C753D
 P 6300 1725
-F 0 "#PWR096" H 6300 1475 50  0001 C CNN
+F 0 "#PWR095" H 6300 1475 50  0001 C CNN
 F 1 "GND" H 6300 1575 50  0000 C CNN
 F 2 "" H 6300 1725 50  0001 C CNN
@@
 	0    -1   -1   0
 $EndComp
+$Comp
+L TEST TP13
+U 1 1 5A9ECA71
+P 4600 1525
+F 0 "TP13" H 4600 1825 50  0000 C BNN
+F 1 "TEST" H 4600 1775 50  0000 C CNN
+F 2 "Measurement_Points:Measurement_Point_Round-SMD-Pad_Small" H 4600 1525 50  0001 C CNN
+F 3 "" H 4600 1525 50  0001 C CNN
+	1    4600 1525
+	1    0    0    -1
+$EndComp
+Wire Wire Line
+	4600 1575 4600 1525
+Connection ~ 4600 1575
+$Comp
+L TEST TP14
+U 1 1 5A9ECB18
+P 4600 3250
+F 0 "TP14" H 4600 3550 50  0000 C BNN
+F 1 "TEST" H 4600 3500 50  0000 C CNN
+F 2 "Measurement_Points:Measurement_Point_Round-SMD-Pad_Small" H 4600 3250 50  0001 C CNN
+F 3 "" H 4600 3250 50  0001 C CNN
+	1    4600 3250
+	1    0    0    -1
+$EndComp
+Wire Wire Line
+	4600 3250 4600 3300
+Connection ~ 4600 3300
+$Comp
+L TEST TP15
+U 1 1 5A9ECBE9
+P 4600 4925
+F 0 "TP15" H 4600 5225 50  0000 C BNN
+F 1 "TEST" H 4600 5175 50  0000 C CNN
+F 2 "Measurement_Points:Measurement_Point_Round-SMD-Pad_Small" H 4600 4925 50  0001 C CNN
+F 3 "" H 4600 4925 50  0001 C CNN
+	1    4600 4925
+	1    0    0    -1
+$EndComp
+Wire Wire Line
+	4600 4975 4600 4925
+Connection ~ 4600 4975
 $EndSCHEMATC

Commit message: Updated PCB
PCB requires mcu to be routed.
Changed to thermistor connector on pcb
Parts:
- renumbered INA6 to INA4, INA4 to INA6
Changed lines of the file:
@@
 Need values for shunt and load resistors\n
 $Comp
-L INA210 INA6
+L INA210 INA4
 U 1 1 5A8C7168
 P 5575 1500
-F 0 "INA6" H 5775 1725 60  0000 C CNN
+F 0 "INA4" H 5775 1725 60  0000 C CNN
 F 1 "INA210" H 5775 1625 60  0000 C CNN
 F 2 "TO_SOT_Packages_SMD:SOT-363_SC-70-6" H 5775 1625 60  0001 C CNN
@@
 $EndComp
 $Comp
-L INA210 INA4
+L INA210 INA6
 U 1 1 5A8C73D5
 P 5425 4900
-F 0 "INA4" H 5625 5125 60  0000 C CNN
+F 0 "INA6" H 5625 5125 60  0000 C CNN
 F 1 "INA210" H 5625 5025 60  0000 C CNN
 F 2 "TO_SOT_Packages_SMD:SOT-363_SC-70-6" H 5625 5025 60  0001 C CNN
